File: hardware/pcb/pcb.kicad_pcb (KiCad board)
At the start: 2 copper layers, 68.6 x 75.3 mm, 55 parts, among them IC1 ATMEGA32U2, P1 USB, P2 PRGM, SW1 SW_PUSH, U00 MX-DI, U01 MX-DI, U02 MX-DI, U03 MX-DI, U10 MX-DI, U11 MX-DI, U12 MX-DI, U13 MX-DI, U20 MX-DI, U21 MX-DI, U22 MX-DI, U23 MX-DI, U30 MX-DI, U32 MX-DI, U33 MX-DI, Y1 HC49S

Commit message: Various PCB edits
Parts:
- IC1: footprint Housings_DFN_QFN:QFN-32-1EP_5x5mm_Pitch0.5mm -> nan-15:QFN-32-1EP_5x5mm_Pitch0.5mm
- moved OSHW 2.38 mm to (157.2, 102.4)
- moved W6 1.19 mm to (169.1, 78.6)
- moved HS1 1.19 mm to (169.1, 131.0)
- renumbered REF*** to OSHW
Routing:
- net /row0: track 220.5 -> 196.1 mm
- net /row3: track 81.6 -> 83.9 mm
- net GND: track 573.5 -> 575.4 mm
- net VCC: track 113.9 -> 115.3 mm
- net /led5: track 88.5 -> 89.9 mm
- net /col1: track 47.7 -> 46.5 mm
Other:
- board size 68.6 x 75.3 mm -> 68.6 x 71.1 mm
- board text added: "SERVICE"
- board text added: "USB"

Commit message: Connect all PWM pins to LEDs; show PCB version number
Parts:
- moved REF*** 2.38 mm to (161.9, 131.0)
Connections:
- IC1 pad 23: /col1 -> /led11
- IC1 pad 26: /led11 -> /col1
- IC1 pad 6: /row2 -> /led0
- IC1 pad 7: /col2 -> /col3
- IC1 pad 8: /col3 -> /col2
- IC1 pad 9: /led0 -> /row2
Routing:
- net /row2: track 64.8 -> 76.2 mm, vias 1 -> 0
- net /col3: track 105.2 -> 95.1 mm
- net /col2: track 88.4 -> 80.9 mm, vias 1 -> 2
- net /led0: track 37.3 -> 32.1 mm
- net /col1: track 46.5 -> 49.5 mm, vias 0 -> 1
- net /led11: track 33.4 -> 30.8 mm
- net /led9: track 17.2 -> 18.3 mm
- net Net-(IC1-Pad24): track 74.2 -> 75.1 mm
- net /led10: track 26.2 -> 25.4 mm
- net /led5: track 89.9 -> 89.3 mm
- net /row0: track 196.1 -> 195.5 mm
- net Net-(C6-Pad2): track 5.04 -> 5.64 mm
- net Net-(IC1-Pad30): track 13.9 -> 13.3 mm
Other:
- board text added: "v0.1"
