File: hardware/pcb/pcb.sch (KiCad schematic (older format))
At the start: 53 parts, among them IC1 ATMEGA32U2, P1 USB, P2 PRGM, SW1 SW_PUSH, U00 MX-DI, U01 MX-DI, U02 MX-DI, U03 MX-DI, U10 MX-DI, U11 MX-DI, U12 MX-DI, U13 MX-DI, U20 MX-DI, U21 MX-DI, U22 MX-DI, U23 MX-DI, U30 MX-DI, U32 MX-DI, U33 MX-DI, Y1 HC49S

Commit message: Various PCB edits
Parts:
- IC1: footprint Housings_DFN_QFN:QFN-32-1EP_5x5mm_Pitch0.5mm -> nan-15:QFN-32-1EP_5x5mm_Pitch0.5mm
Changed lines of the file:
@@
 F 0 "IC1" H 5350 5600 50  0000 C CNN
 F 1 "ATMEGA32U2" H 5350 5500 50  0000 C CNN
-F 2 "Housings_DFN_QFN:QFN-32-1EP_5x5mm_Pitch0.5mm" H 5350 5400 50  0001 C CNN
+F 2 "nan-15:QFN-32-1EP_5x5mm_Pitch0.5mm" H 5350 5400 50  0001 C CNN
 F 3 "http://www.atmel.com/Images/doc7799.pdf" H 6000 2850 50  0001 C CNN
 	1    5900 4300

Commit message: Connect all PWM pins to LEDs; show PCB version number
Parts:
- removed HS1, HS2, HS3, HS4, HS5, HS6, HS7: HEATSINK, nan-15:Plain_Hole_4mm, symbol HEATSINK
Connections:
- net col1: now also IC1.26 ((PCINT10)PC4); no longer IC1.23 ((OC.1A/PCINT8)PC6)
- net col2: now also IC1.8 ((RXD1/AIN1/INT2)PD2); no longer IC1.7 ((AIN0/INT1)PD1)
- net col3: now also IC1.7 ((AIN0/INT1)PD1); no longer IC1.8 ((RXD1/AIN1/INT2)PD2)
- net led0: now also IC1.6 ((OC.0B/INT0)PD0); no longer IC1.9 ((TXD1/INT3)PD3)
- net led11: now also IC1.23 ((OC.1A/PCINT8)PC6); no longer IC1.26 ((PCINT10)PC4)
- net row2: now also IC1.9 ((TXD1/INT3)PD3); no longer IC1.6 ((OC.0B/INT0)PD0)
Changed lines of the file:
@@
 row3
 Text Label 8900 4100 2    60   ~ 0
-row2
+led0
 Text Label 8900 4200 2    60   ~ 0
-col2
+col3
 Text Label 8900 3400 2    60   ~ 0
 row1
@@
 col0
 Text Label 8900 5300 2    60   ~ 0
-col1
+led11
 Text Label 8900 4300 2    60   ~ 0
-col3
+col2
 Text Label 8900 4400 2    60   ~ 0
-led0
+row2
 Text Label 8900 4500 2    60   ~ 0
 led1
@@
 led10
 Text Label 8900 5100 2    60   ~ 0
-led11
+col1
 $Comp
 L CONN_01X06 P2
@@
 	1    0    0    -1
 $EndComp
-$Comp
-L HEATSINK HS1
-U 1 1 5828EBAB
-P 11300 9000
-F 0 "HS1" H 11427 9121 50  0000 L CNN
-F 1 "HEATSINK" H 11427 9030 50  0000 L CNN
-F 2 "nan-15:Plain_Hole_4mm" H 11300 9000 50  0001 C CNN
-F 3 "" H 11300 9000 50  0000 C CNN
-	1    11300 9000
-	1    0    0    -1
-$EndComp
-$Comp
-L HEATSINK HS2
-U 1 1 5828EC7D
-P 11300 9250
-F 0 "HS2" H 11427 9371 50  0000 L CNN
-F 1 "HEATSINK" H 11427 9280 50  0000 L CNN
-F 2 "nan-15:Plain_Hole_4mm" H 11300 9250 50  0001 C CNN
-F 3 "" H 11300 9250 50  0000 C CNN
-	1    11300 9250
-	1    0    0    -1
-$EndComp
-$Comp
-L HEATSINK HS3
-U 1 1 5828F101
-P 12100 9000
-F 0 "HS3" H 12227 9121 50  0000 L CNN
-F 1 "HEATSINK" H 12227 9030 50  0000 L CNN
-F 2 "nan-15:Plain_Hole_4mm" H 12100 9000 50  0001 C CNN
-F 3 "" H 12100 9000 50  0000 C CNN
-	1    12100 9000
-	1    0    0    -1
-$EndComp
-$Comp
-L HEATSINK HS4
-U 1 1 5828F1BB
-P 12100 9250
-F 0 "HS4" H 12227 9371 50  0000 L CNN
-F 1 "HEATSINK" H 12227 9280 50  0000 L CNN
-F 2 "nan-15:Plain_Hole_4mm" H 12100 9250 50  0001 C CNN
-F 3 "" H 12100 9250 50  0000 C CNN
-	1    12100 9250
-	1    0    0    -1
-$EndComp
-$Comp
-L HEATSINK HS5
-U 1 1 5828F261
-P 12900 9000
-F 0 "HS5" H 13027 9121 50  0000 L CNN
-F 1 "HEATSINK" H 13027 9030 50  0000 L CNN
-F 2 "nan-15:Plain_Hole_4mm" H 12900 9000 50  0001 C CNN
-F 3 "" H 12900 9000 50  0000 C CNN
-	1    12900 9000
-	1    0    0    -1
-$EndComp
-$Comp
-L HEATSINK HS6
-U 1 1 5828F2F7
-P 12900 9250
-F 0 "HS6" H 13027 9371 50  0000 L CNN
-F 1 "HEATSINK" H 13027 9280 50  0000 L CNN
-F 2 "nan-15:Plain_Hole_4mm" H 12900 9250 50  0001 C CNN
-F 3 "" H 12900 9250 50  0000 C CNN
-	1    12900 9250
-	1    0    0    -1
-$EndComp
-$Comp
-L HEATSINK HS7
-U 1 1 5828F399
-P 13700 9000
-F 0 "HS7" H 13827 9121 50  0000 L CNN
-F 1 "HEATSINK" H 13827 9030 50  0000 L CNN
-F 2 "nan-15:Plain_Hole_4mm" H 13700 9000 50  0001 C CNN
-F 3 "" H 13700 9000 50  0000 C CNN
-	1    13700 9000
-	1    0    0    -1
-$EndComp

Commit message: Update version numbers on PCB silkscreens
Parts:
- C1, C2, C3, C4, C5, C6: footprint Capacitors_SMD:C_1206_HandSoldering -> Capacitors_SMD:C_1206
- R1, R2, R3, R4: footprint Resistors_SMD:R_1206_HandSoldering -> Resistors_SMD:R_1206
- W0, W1, W10, W11, W2, W3, W4, W5, W50, W51, W52, W53, W6, W7, W8, W9: footprint nan-15:SolderWirePad_single_1-2mmDrill_no_legend -> nan-15:SolderWirePad_2mm_1-2mmDrill_no_legend
- Y1: value HC49S -> MT 16MHz; footprint Crystals:Crystal_HC49-U_Vertical -> nan-15:crystal_MT_32x25; symbol Crystal_Small -> CRYSTAL_SMD
Connections:
- net GND: now also Y1.3 (case)
- net at C4.1, IC1.1 (XTAL1): no longer Y1.1
- net at C5.1, IC1.2 (PC0(XTAL2)): no longer Y1.2
- net D+: now reaches IC1.29 (D+), R2.1
- net D-: now reaches IC1.30 (D-), R3.1
Changed lines of the file:
@@
 Title "NaN-15"
 Date ""
-Rev "0.1"
+Rev "0.2"
 Comp ""
 Comment1 ""
@@
 F 0 "C1" H 2715 1896 50  0000 L CNN
 F 1 "1u" H 2715 1805 50  0000 L CNN
-F 2 "Capacitors_SMD:C_1206_HandSoldering" H 2638 1700 50  0001 C CNN
+F 2 "Capacitors_SMD:C_1206" H 2638 1700 50  0001 C CNN
 F 3 "" H 2600 1850 50  0000 C CNN
 	1    2600 1850
@@
 F 0 "C6" V 4550 4450 50  0000 L CNN
 F 1 "1u" V 4465 4455 50  0000 L CNN
-F 2 "Capacitors_SMD:C_1206_HandSoldering" H 4388 4350 50  0001 C CNN
+F 2 "Capacitors_SMD:C_1206" H 4388 4350 50  0001 C CNN
 F 3 "" H 4350 4500 50  0000 C CNN
 	1    4350 4500
@@
 F 0 "C5" H 4065 4146 50  0000 L CNN
 F 1 "18p" H 4065 4055 50  0000 L CNN
-F 2 "Capacitors_SMD:C_1206_HandSoldering" H 3988 3950 50  0001 C CNN
+F 2 "Capacitors_SMD:C_1206" H 3988 3950 50  0001 C CNN
 F 3 "" H 3950 4100 50  0000 C CNN
 	1    3950 4100
@@
 F 0 "C4" H 3200 4150 50  0000 L CNN
 F 1 "18p" H 3200 4050 50  0000 L CNN
-F 2 "Capacitors_SMD:C_1206_HandSoldering" H 3488 3950 50  0001 C CNN
+F 2 "Capacitors_SMD:C_1206" H 3488 3950 50  0001 C CNN
 F 3 "" H 3450 4100 50  0000 C CNN
 	1    3450 4100
@@
 $EndComp
 $Comp
-L Crystal_Small Y1
+L CRYSTAL_SMD Y1
 U 1 1 58276AB3
 P 3700 3900
 F 0 "Y1" H 3700 4100 50  0000 C CNN
-F 1 "HC49S" H 3700 4034 50  0000 C CNN
-F 2 "Crystals:Crystal_HC49-U_Vertical" H 3700 3900 50  0001 C CNN
+F 1 "MT 16MHz" H 3700 4034 50  0000 C CNN
+F 2 "nan-15:crystal_MT_32x25" H 3700 3900 50  0001 C CNN
 F 3 "" H 3700 3900 50  0000 C CNN
 	1    3700 3900
@@
 F 0 "R3" V 2950 4800 50  0000 C CNN
 F 1 "22" V 2900 4950 50  0000 C CNN
-F 2 "Resistors_SMD:R_1206_HandSoldering" H 2950 4800 50  0001 C CNN
+F 2 "Resistors_SMD:R_1206" H 2950 4800 50  0001 C CNN
 F 3 "" H 2950 4800 50  0000 C CNN
 	1    2950 4800
@@
 F 0 "R2" V 2950 4700 50  0000 C CNN
 F 1 "22" V 2900 4850 50  0000 C CNN
-F 2 "Resistors_SMD:R_1206_HandSoldering" H 2950 4700 50  0001 C CNN
+F 2 "Resistors_SMD:R_1206" H 2950 4700 50  0001 C CNN
 F 3 "" H 2950 4700 50  0000 C CNN
 	1    2950 4700
@@
 F 0 "R1" H 3359 3246 50  0000 L CNN
 F 1 "10k" H 3359 3155 50  0000 L CNN
-F 2 "Resistors_SMD:R_1206_HandSoldering" H 3300 3200 50  0001 C CNN
+F 2 "Resistors_SMD:R_1206" H 3300 3200 50  0001 C CNN
 F 3 "" H 3300 3200 50  0000 C CNN
 	1    3300 3200
@@
 F 0 "C2" H 3215 1896 50  0000 L CNN
 F 1 "100n" H 3215 1805 50  0000 L CNN
-F 2 "Capacitors_SMD:C_1206_HandSoldering" H 3138 1700 50  0001 C CNN
+F 2 "Capacitors_SMD:C_1206" H 3138 1700 50  0001 C CNN
 F 3 "" H 3100 1850 50  0000 C CNN
 	1    3100 1850
@@
 F 0 "C3" H 3665 1896 50  0000 L CNN
 F 1 "100n" H 3665 1805 50  0000 L CNN
-F 2 "Capacitors_SMD:C_1206_HandSoldering" H 3588 1700 50  0001 C CNN
+F 2 "Capacitors_SMD:C_1206" H 3588 1700 50  0001 C CNN
 F 3 "" H 3550 1850 50  0000 C CNN
 	1    3550 1850
@@
 F 0 "R4" V 7100 4800 50  0000 C CNN
 F 1 "10k" V 7050 4950 50  0000 C CNN
-F 2 "Resistors_SMD:R_1206_HandSoldering" H 7100 4800 50  0001 C CNN
+F 2 "Resistors_SMD:R_1206" H 7100 4800 50  0001 C CNN
 F 3 "" H 7100 4800 50  0000 C CNN
 	1    7100 4800
@@
 F 0 "W0" V 9400 8538 50  0000 L CNN
 F 1 "TEST_1P" V 9445 8538 50  0001 L CNN
-F 2 "nan-15:SolderWirePad_single_1-2mmDrill_no_legend" H 9600 8350 50  0001 C CNN
+F 2 "nan-15:SolderWirePad_2mm_1-2mmDrill_no_legend" H 9600 8350 50  0001 C CNN
 F 3 "" H 9600 8350 50  0000 C CNN
 	1    9400 8350
@@
 F 0 "W1" V 9400 8638 50  0000 L CNN
 F 1 "TEST_1P" V 9445 8638 50  0001 L CNN
-F 2 "nan-15:SolderWirePad_single_1-2mmDrill_no_legend" H 9600 8450 50  0001 C CNN
+F 2 "nan-15:SolderWirePad_2mm_1-2mmDrill_no_legend" H 9600 8450 50  0001 C CNN
 F 3 "" H 9600 8450 50  0000 C CNN
 	1    9400 8450
@@
 F 0 "W2" V 9400 8738 50  0000 L CNN
 F 1 "TEST_1P" V 9445 8738 50  0001 L CNN
-F 2 "nan-15:SolderWirePad_single_1-2mmDrill_no_legend" H 9600 8550 50  0001 C CNN
+F 2 "nan-15:SolderWirePad_2mm_1-2mmDrill_no_legend" H 9600 8550 50  0001 C CNN
 F 3 "" H 9600 8550 50  0000 C CNN
 	1    9400 8550
@@
 F 0 "W3" V 9400 8838 50  0000 L CNN
 F 1 "TEST_1P" V 9445 8838 50  0001 L CNN
-F 2 "nan-15:SolderWirePad_single_1-2mmDrill_no_legend" H 9600 8650 50  0001 C CNN
+F 2 "nan-15:SolderWirePad_2mm_1-2mmDrill_no_legend" H 9600 8650 50  0001 C CNN
 F 3 "" H 9600 8650 50  0000 C CNN
 	1    9400 8650
@@
 F 0 "W4" V 9400 8938 50  0000 L CNN
 F 1 "TEST_1P" V 9445 8938 50  0001 L CNN
-F 2 "nan-15:SolderWirePad_single_1-2mmDrill_no_legend" H 9600 8750 50  0001 C CNN
+F 2 "nan-15:SolderWirePad_2mm_1-2mmDrill_no_legend" H 9600 8750 50  0001 C CNN
 F 3 "" H 9600 8750 50  0000 C CNN
 	1    9400 8750
@@
 F 0 "W5" V 9400 9038 50  0000 L CNN
 F 1 "TEST_1P" V 9445 9038 50  0001 L CNN
-F 2 "nan-15:SolderWirePad_single_1-2mmDrill_no_legend" H 9600 8850 50  0001 C CNN
+F 2 "nan-15:SolderWirePad_2mm_1-2mmDrill_no_legend" H 9600 8850 50  0001 C CNN
 F 3 "" H 9600 8850 50  0000 C CNN
 	1    9400 8850
@@
 F 0 "W6" V 9400 9138 50  0000 L CNN
 F 1 "TEST_1P" V 9445 9138 50  0001 L CNN
-F 2 "nan-15:SolderWirePad_single_1-2mmDrill_no_legend" H 9600 8950 50  0001 C CNN
+F 2 "nan-15:SolderWirePad_2mm_1-2mmDrill_no_legend" H 9600 8950 50  0001 C CNN
 F 3 "" H 9600 8950 50  0000 C CNN
 	1    9400 8950
@@
 F 0 "W7" V 9400 9238 50  0000 L CNN
 F 1 "TEST_1P" V 9445 9238 50  0001 L CNN
-F 2 "nan-15:SolderWirePad_single_1-2mmDrill_no_legend" H 9600 9050 50  0001 C CNN
+F 2 "nan-15:SolderWirePad_2mm_1-2mmDrill_no_legend" H 9600 9050 50  0001 C CNN
 F 3 "" H 9600 9050 50  0000 C CNN
 	1    9400 9050
@@
 F 0 "W8" V 9400 9338 50  0000 L CNN
 F 1 "TEST_1P" V 9445 9338 50  0001 L CNN
-F 2 "nan-15:SolderWirePad_single_1-2mmDrill_no_legend" H 9600 9150 50  0001 C CNN
+F 2 "nan-15:SolderWirePad_2mm_1-2mmDrill_no_legend" H 9600 9150 50  0001 C CNN
 F 3 "" H 9600 9150 50  0000 C CNN
 	1    9400 9150
@@
 F 0 "W9" V 9400 9438 50  0000 L CNN
 F 1 "TEST_1P" V 9445 9438 50  0001 L CNN
-F 2 "nan-15:SolderWirePad_single_1-2mmDrill_no_legend" H 9600 9250 50  0001 C CNN
+F 2 "nan-15:SolderWirePad_2mm_1-2mmDrill_no_legend" H 9600 9250 50  0001 C CNN
 F 3 "" H 9600 9250 50  0000 C CNN
 	1    9400 9250
@@
 F 0 "W10" V 9400 9537 50  0000 L CNN
 F 1 "TEST_1P" V 9445 9538 50  0001 L CNN
-F 2 "nan-15:SolderWirePad_single_1-2mmDrill_no_legend" H 9600 9350 50  0001 C CNN
+F 2 "nan-15:SolderWirePad_2mm_1-2mmDrill_no_legend" H 9600 9350 50  0001 C CNN
 F 3 "" H 9600 9350 50  0000 C CNN
 	1    9400 9350
@@
 F 0 "W11" V 9400 9637 50  0000 L CNN
 F 1 "TEST_1P" V 9445 9638 50  0001 L CNN
-F 2 "nan-15:SolderWirePad_single_1-2mmDrill_no_legend" H 9600 9450 50  0001 C CNN
+F 2 "nan-15:SolderWirePad_2mm_1-2mmDrill_no_legend" H 9600 9450 50  0001 C CNN
 F 3 "" H 9600 9450 50  0000 C CNN
 	1    9400 9450
@@
 F 0 "W50" V 6700 8537 50  0000 L CNN
 F 1 "TEST_1P" V 6745 8538 50  0001 L CNN
-F 2 "nan-15:SolderWirePad_single_1-2mmDrill_no_legend" H 6900 8350 50  0001 C CNN
+F 2 "nan-15:SolderWirePad_2mm_1-2mmDrill_no_legend" H 6900 8350 50  0001 C CNN
 F 3 "" H 6900 8350 50  0000 C CNN
 	1    6700 8350
@@
 F 0 "W51" V 6700 8837 50  0000 L CNN
 F 1 "TEST_1P" V 6745 8838 50  0001 L CNN
-F 2 "nan-15:SolderWirePad_single_1-2mmDrill_no_legend" H 6900 8650 50  0001 C CNN
+F 2 "nan-15:SolderWirePad_2mm_1-2mmDrill_no_legend" H 6900 8650 50  0001 C CNN
 F 3 "" H 6900 8650 50  0000 C CNN
 	1    6700 8650
@@
 F 0 "W52" V 6700 9137 50  0000 L CNN
 F 1 "TEST_1P" V 6745 9138 50  0001 L CNN
-F 2 "nan-15:SolderWirePad_single_1-2mmDrill_no_legend" H 6900 8950 50  0001 C CNN
+F 2 "nan-15:SolderWirePad_2mm_1-2mmDrill_no_legend" H 6900 8950 50  0001 C CNN
 F 3 "" H 6900 8950 50  0000 C CNN
 	1    6700 8950
@@
 F 0 "W53" V 6700 9437 50  0000 L CNN
 F 1 "TEST_1P" V 6745 9438 50  0001 L CNN
-F 2 "nan-15:SolderWirePad_single_1-2mmDrill_no_legend" H 6900 9250 50  0001 C CNN
+F 2 "nan-15:SolderWirePad_2mm_1-2mmDrill_no_legend" H 6900 9250 50  0001 C CNN
 F 3 "" H 6900 9250 50  0000 C CNN
 	1    6700 9250
@@
 	0    -1   -1   0
 $EndComp
+$Comp
+L GND #PWR028
+U 1 1 583F1710
+P 3700 4000
+F 0 "#PWR028" H 3700 3750 50  0001 C CNN
+F 1 "GND" H 3705 3827 50  0000 C CNN
+F 2 "" H 3700 4000 50  0000 C CNN
+F 3 "" H 3700 4000 50  0000 C CNN
+	1    3700 4000
+	1    0    0    -1
+$EndComp
+Text Label 3650 4700 0    60   ~ 0
+D+
+Text Label 3650 4800 0    60   ~ 0
+D-
 $EndSCHEMATC
